Commit message: sine_function

File: src/mini_challenge_2/urdf/dc_motor.urdf (robot description, URDF)
Before this commit: robot single_link_arm, 2 links, 1 joints
Links:
- added link Motor; collision box size=0.1 0.1 0.1; visual mesh filename=package://mini_challenge_2/models/Motor.stl scale=1 1 1
- link Wheel: geometry collision cylinder length=0.05 radius=0.1; visual mesh filename=package://mini_challenge_2/models/Llanta.stl scale=1 1 1
Joints:
- added joint joint1: type fixed, parent world, child Motor, origin xyz=0 0 1 rpy=0 0 0
- joint joint2: parent world -> Motor

Commit message: urdf

File: src/mini_challenge_2/urdf/dc_motor.urdf (robot description, URDF)
Before this commit: robot single_link_arm, 3 links, 2 joints
Joints:
- joint joint2: axis 1 0 0 -> 0 0 1
